File: Make Files/CAN_Firewall.kicad_pcb (KiCad board)
At the start: 2 copper layers, 50.1 x 23.8 mm, 32 parts, among them J1 DB9, J2 DB9, U1 MCP2551-I/SN, U2 MCP2551-I/SN, U3 MC78M05CDT, U4 AT32UC3C, U5 PESDxL5UY

Commit message: Version 1.1 Produced
Moved in from archive
Parts:
- removed 12V: PINHEAD1-2, Connect:PINHEAD1-2
- added C14: 100N, Custom Parts:R_0603_sm, F.Cu at (53.5, 133.5)
- added CON1: BARREL_JACK, Connect:BARREL_JACK, F.Cu at (85.3, 118.0)
- added CON2: AVR-JTAG-10, Socket_Strips:Socket_Strip_Straight_2x05, F.Cu at (74.8, 125.0)
- added CON3: AVR-AW-6, Socket_Strips:Socket_Strip_Straight_2x03, F.Cu at (69.8, 117.1)
- added D2: BLUE, Custom Parts:Diode_0805_12, F.Cu at (105.0, 120.0)
- added D4: RED, Custom Parts:Diode_0805_12, F.Cu at (83.0, 135.0)
- added D5: BLUE, Custom Parts:Diode_0805_12, F.Cu at (83.0, 132.0)
- added D6: BLUE, Custom Parts:Diode_0805_12, F.Cu at (75.5, 114.0)
- added F2: FUSE, Custom Parts:R_1210_SM, F.Cu at (93.5, 115.5)
- added F3: FUSE, Custom Parts:R_1210_SM, F.Cu at (44.0, 126.5)
- added FB1: 220, Custom Parts:Diode_0805_12_SM, F.Cu at (49.5, 127.0)
- added FB2: 220, Custom Parts:Diode_0805_12_SM, F.Cu at (93.5, 119.0)
- added J3: DB9, Connect:DB9F_CI, B.Cu at (108.0, 142.5)
- added P1: USB_OTG, Custom Parts:USB_Micro-B-DX4R005JJ2R1800, F.Cu at (47.0, 111.5)
- added P2: USB_OTG, Custom Parts:USB_Micro-B-DX4R005JJ2R1800, F.Cu at (101.0, 111.5)
- added P3: DIAG Port, Socket_Strips:Socket_Strip_Straight_1x12, F.Cu at (88.6, 152.2)
- added R10: 470, Custom Parts:R_0603_sm, F.Cu at (105.0, 130.5)
- added R11: 470, Custom Parts:R_0603_sm, F.Cu at (105.0, 133.5)
- added R12: 470, Custom Parts:R_0603_sm, F.Cu at (43.5, 131.5)
- added R13: 470, Custom Parts:R_0603_sm, F.Cu at (87.5, 135.0)
- added R14: 470, Custom Parts:R_0603_sm, F.Cu at (87.5, 132.0)
- added R15: 470, Custom Parts:R_0603_sm, F.Cu at (75.5, 117.5)
- added SW1: SPST, Custom Parts:SW_SPST_FSMSM_SM, F.Cu at (101.0, 152.0)
- added U6: MCP25625, Housings_SSOP:SSOP-28_5.3x10.2mm_Pitch0.65mm, F.Cu at (94.6, 139.9)
- added X1: TXC, Custom Parts:TXC, F.Cu at (61.5, 133.0)
- C1, C2: value 560P -> 10N; footprint cUSTOM pARTS:R_0603_sm -> Custom Parts:R_0603_sm
- C10, C11, C12, C13, C8, C9, R8: footprint cUSTOM pARTS:R_0603_sm -> Custom Parts:R_0603_sm
- C3, C4: value 560P -> 100N; footprint cUSTOM pARTS:R_0603_sm -> Custom Parts:R_0603_sm
- C5: value 10N -> 100N; footprint cUSTOM pARTS:R_0603_sm -> Custom Parts:R_0603_sm
- C6: value 4U7 -> 10N; footprint Capacitors_Tantalum_SMD:TantalC_SizeA_EIA-3216_Reflow -> Custom Parts:R_0603_sm
- C7: value 100N -> 4U7; footprint cUSTOM pARTS:R_0603_sm -> Capacitors_Tantalum_SMD:TantalC_SizeA_EIA-3216_Reflow
- D1: value SMBJ16A -> RED; footprint Diodes_SMD:Diode-SMB_Standard -> Custom Parts:Diode_0805_12
- F1: footprint cUSTOM pARTS:R_1210_SM -> Custom Parts:R_1210_SM
- J1: value DB9 -> +5V_SRC; footprint Connect:DB9F_CI -> Socket_Strips:Socket_Strip_Straight_1x03
- R1: value 470 -> 22; footprint cUSTOM pARTS:R_0603_sm -> Custom Parts:R_0603_sm
- R2, R3: value 100 -> 22; footprint cUSTOM pARTS:R_0603_sm -> Custom Parts:R_0603_sm
- R4, R5: value 100 -> DNS; footprint cUSTOM pARTS:R_0603_sm -> Custom Parts:R_0603_sm
- R6, R7: value 4K7 -> 470; footprint cUSTOM pARTS:R_0603_sm -> Custom Parts:R_0603_sm
- R9: value 470 -> 4K7
- U1: value MCP2551-I/SN -> AT32UC3C; footprint Power_Integrations:SO-8 -> Housings_QFP:LQFP-64_10x10mm_Pitch0.5mm
- U2: value MCP2551-I/SN -> FT232RL-SSOP; footprint Power_Integrations:SO-8 -> Housings_SSOP:SSOP-28_5.3x10.2mm_Pitch0.65mm
- U4: value AT32UC3C -> SMF05; footprint Housings_QFP:LQFP-64_10x10mm_Pitch0.5mm -> Housings_SOT-23_SOT-143_TSOT-6:SC-70-6
- U5: value PESDxL5UY -> MCP25625; footprint Housings_SOT-23_SOT-143_TSOT-6:SC-70-6 -> Housings_SSOP:SSOP-28_5.3x10.2mm_Pitch0.65mm
- moved U4 122.1 mm to (93.0, 152.0), turned to 180 degrees
- moved J2 117.6 mm to (40.0, 142.5), turned to 90 degrees
- moved D1 117.1 mm to (105.0, 125.5), turned to 0 degrees
- moved C5 116.9 mm to (61.5, 139.0), turned to 180 degrees
- moved U5 116.8 mm to (53.5, 141.5), turned to 0 degrees
- moved R6 115.9 mm to (84.5, 144.0), turned to 180 degrees
- moved R4 115.9 mm to (66.0, 146.5), turned to 180 degrees
- moved R1 115.0 mm to (66.0, 144.0), turned to 180 degrees
- moved C9 114.8 mm to (97.2, 147.2), turned to 180 degrees
- moved R7 113.3 mm to (84.5, 146.5), turned to 180 degrees
- moved R3 112.2 mm to (61.5, 141.5), turned to 180 degrees
- moved C10 111.7 mm to (71.2, 146.5), turned to 0 degrees
- moved R5 109.6 mm to (61.5, 144.0), turned to 0 degrees
- moved C6 107.3 mm to (43.6, 134.0), turned to 0 degrees
- moved C12 107.2 mm to (84.5, 141.5), turned to 0 degrees
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Connections:
- C12 pad 1: Net-(C12-Pad1) -> +5V
- C13 pad 1: Net-(C13-Pad1) -> +5V
- C4 pad 1: Net-(C4-Pad1) -> +3V3
- C5 pad 1: +12V -> Net-(C5-Pad1)
- C6 pad 1: Net-(C6-Pad1) -> +12V
- C7 pad 1: Net-(C6-Pad1) -> Net-(C7-Pad1)
- C8 pad 1: +5V -> Net-(C7-Pad1)
- D1 pad 1: +12V -> Net-(D1-Pad1)
- D1 pad 2: GND -> Net-(D1-Pad2)
- F1 pad 1: +12V -> Net-(F1-Pad1)
- F1 pad 2: Net-(C6-Pad1) -> Net-(C1-Pad1)
- J1 pad 1: 5P -> USB5
- J1 pad 2: IVI_CANL -> +5V
- J1 pad 3: GND -> VBUS
- J2 pad 1: Net-(J2-Pad1) -> ~RESET/A_DATA
- J2 pad 2: CAR_CANL -> IVI_CANL
- J2 pad 7: CAR_CANH -> IVI_CANH
- R1 pad 1: +5V -> CLK1
- R1 pad 2: 5P -> Net-(R1-Pad2)
- R2 pad 1: IVI_CANH -> CLK2
- R2 pad 2: Net-(C1-Pad1) -> Net-(R1-Pad2)
- R3 pad 1: IVI_CANL -> CLK3
- R3 pad 2: Net-(C2-Pad1) -> Net-(R1-Pad2)
- R4 pad 1: CAR_CANL -> CLK1
- R4 pad 2: Net-(C3-Pad1) -> CLK3_OUT
- R5 pad 1: CAR_CANH -> CLK3
- R5 pad 2: Net-(C4-Pad1) -> CLK2_OUT
- R6 pad 1: Net-(R6-Pad1) -> LOOP_B
- R6 pad 2: GND -> Net-(R6-Pad2)
- R7 pad 1: Net-(R7-Pad1) -> LOOP_A
- R7 pad 2: GND -> Net-(R7-Pad2)
- R8 pad 1: Net-(J2-Pad6) -> Net-(R8-Pad1)
- R8 pad 2: LOOP_A -> USB5
- R9 pad 1: Net-(J2-Pad1) -> Net-(R8-Pad1)
- R9 pad 2: LOOP_B -> GND
- U1 pad 1: TX0 -> TCK
- U1 pad 2: GND -> TDI
- U1 pad 3: +5V -> TDO
- U1 pad 4: RX0 -> TMS
- U1 pad 5: Net-(U1-Pad5) -> +5V
- U1 pad 6: IVI_CANL -> GND
- U1 pad 7: IVI_CANH -> Net-(U1-Pad7)
- U1 pad 8: Net-(R6-Pad1) -> Net-(U1-Pad8)
- U2 pad 1: TX1 -> RX_DBG
- U2 pad 2: GND -> Net-(U2-Pad2)
- U2 pad 3: +5V -> Net-(U2-Pad3)
- U2 pad 4: RX1 -> +5V
- U2 pad 5: Net-(U2-Pad5) -> TX_DBG
- U2 pad 6: CAR_CANL -> Net-(U2-Pad6)
- U2 pad 7: CAR_CANH -> GND
- U2 pad 8: Net-(R7-Pad1) -> (no net)
- U3 pad 1: Net-(C6-Pad1) -> Net-(C7-Pad1)
- U4 pad 1: Net-(U4-Pad1) -> LOOP_A
- U4 pad 2: Net-(U4-Pad2) -> GND
- U4 pad 3: A_DATAOUT -> Net-(U4-Pad3)
- U4 pad 4: +5V -> ~RESET/A_DATA
- U4 pad 5: (no net) -> Net-(U4-Pad5)
- U4 pad 6: GND -> LOOP_B
- U5 pad 1: LOOP_A -> +5V
- U5 pad 2: GND -> Net-(U5-Pad2)
- U5 pad 3: 5P -> IVI_CANH
- U5 pad 4: ~RESET/A_DATA -> IVI_CANL
- U5 pad 5: A_DATAOUT -> IVI_STBY
- U5 pad 6: LOOP_B -> IVI_Tx1RTS
Routing:
- net +5V: track 58.2 -> 224.4 mm, vias 0 -> 7
- net GND: track 156.9 -> 305.4 mm, vias 37 -> 58
- net ~RESET/A_DATA: track 33.7 -> 102.8 mm, vias 3 -> 4
- net CLK2_OUT: track 0.00 -> 65.7 mm, vias 0 -> 4
- net SCLK: track 0.00 -> 62.3 mm, vias 0 -> 7
- net MOSI: track 0.00 -> 53.3 mm, vias 0 -> 1
- net MISO: track 0.00 -> 50.0 mm, vias 0 -> 1
- net USBM: track 0.00 -> 44.3 mm, vias 0 -> 2
- net USBP: track 0.00 -> 43.8 mm, vias 0 -> 2
- net IVI_STBY: track 0.00 -> 43.8 mm, vias 0 -> 2
- net USB5: track 0.00 -> 43.5 mm, vias 0 -> 2
- net +12V: track 68.9 -> 111.7 mm, vias 2 -> 4
- net TX_DBG: track 0.00 -> 41.8 mm, vias 0 -> 3
- net RX_DBG: track 0.00 -> 41.8 mm, vias 0 -> 3
- net RX0: track 37.4 -> 0.00 mm, vias 2 -> 0
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- added copper zone on F.Cu, net Net-(C7-Pad1)
Other:
- board size 50.1 x 23.8 mm -> 68 x 44 mm
- board text added: "+12V"
- board text added: "+5V SOURCE USE ONLY ONE NC FOR +12V"
- board text added: "A-WIRE"
- board text added: "BOOT"
- board text added: "IVI CAN"
- board text added: "I_RX I_TX MOSI MISO SCLK ICS CCS RXD TXD C_TX C_RX GND"
- board text added: "JTAG"
- board text added: "Jaguar Land Rovver CANBUS Firewall V1.1 Open Source Hardware Jesse Banks 2015"
- board text added: "LOOP JUMPER"
- board text added: "PWR"
- board text added: "RX"
- board text added: "SERIAL DEBUG"
- board text added: "TX"
- board text added: "USB BOOT +12V DEBUG USB"
- board text removed: "- + 12V"
- board text removed: "AVR PROG"
- board text removed: "CANBUS Firewall V1.1 Open Source Hardware Jaguar Land Rover OSTC Jesse Banks 2015"
- board text removed: "CAR"
- board text removed: "IVI"
- board text removed: "Unlabeled C's are 100N"

Commit message: Active project import
moved from archive
Parts:
- added D3: SMBJ16A, Diodes_SMD:SMB_Handsoldering, F.Cu at (75.4, 116.5)
- added JP1: Matrix A, Connect:GS3, B.Cu at (94.5, 150.0)
- added JP10: Matrix E, Connect:GS3, B.Cu at (100.0, 143.5)
- added JP2: Matrix B, Connect:GS3, B.Cu at (94.5, 140.5)
- added JP3: Matrix C, Connect:GS3, B.Cu at (94.5, 137.5)
- added JP4: Matrix D, Connect:GS3, B.Cu at (94.5, 147.0)
- added JP5: Matrix E, Connect:GS3, B.Cu at (94.5, 143.5)
- added JP6: Matrix A, Connect:GS3, B.Cu at (100.0, 150.0)
- added JP7: Matrix B, Connect:GS3, B.Cu at (100.0, 140.5)
- added JP8: Matrix C, Connect:GS3, B.Cu at (100.0, 137.5)
- added JP9: Matrix D, Connect:GS3, B.Cu at (100.0, 147.0)
- added R16: 0, Custom Parts:R_0603_sm, F.Cu at (51.5, 151.5)
- added R17: 0, Custom Parts:R_0603_sm, F.Cu at (92.5, 153.5)
- added R18: 0, Custom Parts:R_0603_sm, F.Cu at (51.5, 149.0)
- added R19: 0, Custom Parts:R_0603_sm, F.Cu at (92.5, 151.5)
- added R20: 120, Custom Parts:R_0603_sm, F.Cu at (53.0, 130.0)
- added R21: 120, Custom Parts:R_0603_sm, F.Cu at (89.5, 133.5)
- added REF**: MountingHole_3-5mm, Mounting_Holes:MountingHole_3-5mm, F.Cu at (95.5, 159.0)
- added REF**: MountingHole_3-5mm, Mounting_Holes:MountingHole_3-5mm, F.Cu at (50.5, 159.1)
- added REF**: MountingHole_3-5mm, Mounting_Holes:MountingHole_3-5mm, F.Cu at (50.5, 109.0)
- added REF**: Symbol_OSHW-Logo_SilkScreen_BIG, Symbols:Symbol_OSHW-Logo_SilkScreen_BIG, B.Cu at (96.1, 98.8)
- added REF**: MountingHole_3-5mm, Mounting_Holes:MountingHole_3-5mm, F.Cu at (95.5, 109.0)
- added SW2: SPST, Custom Parts:SW_SPST_FSMSM_SM, F.Cu at (48.0, 133.5)
- added SW3: SPST, Custom Parts:SW_SPST_FSMSM_SM, F.Cu at (100.5, 133.5)
- C7: value 4U7 -> 47U; footprint Capacitors_Tantalum_SMD:TantalC_SizeA_EIA-3216_Reflow -> Capacitors_SMD:c_elec_6.3x5.3
- CON2: footprint Socket_Strips:Socket_Strip_Straight_2x05 -> Pin_Headers:Pin_Header_Straight_2x05
- CON3: footprint Socket_Strips:Socket_Strip_Straight_2x03 -> Pin_Headers:Pin_Header_Straight_2x03
- D1: value RED -> YELLOW
- D2: value BLUE -> WHITE
- D5: value BLUE -> GREEN
- J1: footprint Socket_Strips:Socket_Strip_Straight_1x03 -> Pin_Headers:Pin_Header_Straight_1x03
- P3: footprint Socket_Strips:Socket_Strip_Straight_1x12 -> Pin_Headers:Pin_Header_Straight_1x12
- R4, R5: value DNS -> 470
- moved R12 52.3 mm to (95.0, 140.5), turned to 180 degrees
- moved C14 35.4 mm to (87.5, 123.5)
- moved C11 34.4 mm to (60.0, 129.5), turned to 0 degrees
- moved R5 31.6 mm to (87.5, 126.0)
- moved R4 28.0 mm to (87.5, 128.5), turned to 0 degrees
- moved R11 17.5 mm to (98.0, 117.5)
- moved F2 17.4 mm to (105.0, 128.5), turned to 90 degrees
- moved R10 17.4 mm to (93.5, 117.5), turned to 0 degrees
- moved D1 15.9 mm to (93.5, 114.5), turned to 180 degrees
- moved FB2 14.2 mm to (83.0, 128.5), turned to 0 degrees
- moved C1 11.1 mm to (43.9, 130.0), turned to 0 degrees
- moved CON2 9.81 mm to (65.0, 125.5), turned to 90 degrees
- moved C2 8.90 mm to (105.0, 124.5)
- moved D2 8.90 mm to (98.0, 114.5)
- moved C5 8.14 mm to (60.0, 147.0)
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Connections:
- C14 pad 1: +5V -> USB5
- J2 pad 1: ~RESET/A_DATA -> Net-(J2-Pad1)
- J2 pad 5: GND -> Net-(J2-Pad5)
- J3 pad 1: LOOP_B -> A
- J3 pad 4: Net-(J3-Pad4) -> B
- J3 pad 5: GND -> C
- J3 pad 6: LOOP_A -> D
- J3 pad 8: Net-(J3-Pad8) -> E
- P3 pad 10: MOSI -> IVI_CS
- P3 pad 2: CAR_RxCAN -> RX_DBG
- P3 pad 3: CAR_TxCAN -> TX_DBG
- P3 pad 4: TX_DBG -> CAR_CS
- P3 pad 5: RX_DBG -> SCLK
- P3 pad 6: CAR_CS -> MISO
- P3 pad 7: IVI_CS -> MOSI
- P3 pad 8: SCLK -> CAR_TxCAN
- P3 pad 9: MISO -> CAR_RxCAN
- R10 pad 2: +5V -> USB5
- R11 pad 2: +5V -> USB5
- R12 pad 1: Net-(J2-Pad6) -> Net-(JP10-Pad1)
- R4 pad 1: CLK1 -> RX_DBG
- R4 pad 2: CLK3_OUT -> Net-(R4-Pad2)
- R5 pad 1: CLK3 -> TX_DBG
- R5 pad 2: CLK2_OUT -> Net-(R5-Pad2)
- U1 pad 39: Net-(U1-Pad39) -> IVI_RxCAN
- U1 pad 40: IVI_CS -> IVI_TxCAN
- U1 pad 41: Net-(U1-Pad41) -> IVI_CS
- U1 pad 43: Net-(U1-Pad43) -> Net-(R7-Pad2)
- U1 pad 44: Net-(U1-Pad44) -> Net-(R6-Pad2)
- U1 pad 45: Net-(R7-Pad2) -> CAR_RxCAN
- U1 pad 46: Net-(R6-Pad2) -> CAR_TxCAN
- U1 pad 57: CAR_INT -> Net-(U1-Pad57)
- U1 pad 58: Net-(U1-Pad58) -> LED1
- U1 pad 59: Net-(U1-Pad59) -> LED2
- U1 pad 60: Net-(U1-Pad60) -> CAR_INT
- U1 pad 62: LED1 -> Net-(U1-Pad62)
- U1 pad 63: LED2 -> Net-(U1-Pad63)
- U2 pad 1: RX_DBG -> Net-(R4-Pad2)
- U2 pad 20: +5V -> USB5
- U2 pad 4: +5V -> USB5
- U2 pad 5: TX_DBG -> Net-(R5-Pad2)
- U5 pad 20: IVI_TxCAN -> Net-(R18-Pad2)
- U5 pad 21: IVI_RxCAN -> Net-(R16-Pad2)
- U5 pad 3: IVI_CANH -> IVI_CANL
- U5 pad 4: IVI_CANL -> IVI_CANH
- U6 pad 20: CAR_TxCAN -> Net-(R19-Pad2)
- U6 pad 21: CAR_RxCAN -> Net-(R17-Pad2)
- U6 pad 3: CAR_CANH -> CAR_CANL
- U6 pad 4: CAR_CANL -> CAR_CANH
Routing:
- net GND: track 305.4 -> 418.1 mm, vias 58 -> 69
- net CLK2_OUT: track 65.7 -> 0.00 mm, vias 4 -> 0
- net +5V: track 224.4 -> 183.2 mm, vias 7 -> 4
- net USB5: track 43.5 -> 70.0 mm
- net Net-(F2-Pad1): track 3.71 -> 29.8 mm
- net IVI_TxCAN: track 20.6 -> 46.7 mm, vias 0 -> 1
- net IVI_RxCAN: track 23.9 -> 46.9 mm, vias 2 -> 1
- net CAR_TxCAN: track 21.5 -> 42.2 mm, vias 0 -> 2
- net CAR_CANL: track 18.0 -> 38.6 mm, vias 1 -> 3
- net CAR_RxCAN: track 24.2 -> 44.5 mm, vias 0 -> 2
- net IVI_CANH: track 11.1 -> 31.3 mm, vias 1 -> 2
- net IVI_CANL: track 14.0 -> 32.1 mm, vias 0 -> 2
- net CAR_CANH: track 16.4 -> 34.3 mm, vias 0 -> 2
- net Net-(R21-Pad1): track 0.00 -> 17.6 mm
- net Net-(J2-Pad6): track 20.2 -> 3.44 mm, vias 1 -> 0
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- added copper zone on F.Cu, net Net-(C2-Pad1)
Other:
- board size 68 x 44 mm -> 68 x 58 mm
- board text added: "120ohm Terminator"
- board text added: "A/B LOOP JUMPER"
- board text added: "AVR BOOT"
- board text added: "BOOT USB REG. +12V DEBUG USB"
- board text added: "CAR CAN"
- board text added: "GND"
- board text added: "I_RX I_TX ICS C_RX C_TX MOSI MISO SCLK CCS TXD RXD GND"
- board text added: "Jaguar Land Rover CANBUS Firewall V1.2 Open Source Hardware Jesse Banks 2016"
- board text added: "LED1 RED"
- board text added: "LED2 GREEN"
- board text added: "LOOP-A LOOP-B V-REF A-DATA"
- board text added: "PIN-5 PIN-4 PIN-8 PIN-6 PIN-1"
- board text added: "Power"
- board text removed: "BOOT"
- board text removed: "I_RX I_TX MOSI MISO SCLK ICS CCS RXD TXD C_TX C_RX GND"
- board text removed: "Jaguar Land Rovver CANBUS Firewall V1.1 Open Source Hardware Jesse Banks 2015"
- board text removed: "LOOP JUMPER"
- board text removed: "PWR"
- board text removed: "USB BOOT +12V DEBUG USB"
