File: Make Files/CAN_Firewall.sch (KiCad schematic (older format))
At the start: 32 parts, among them J1 DB9, J2 DB9, U1 MCP2551-I/SN, U2 MCP2551-I/SN, U3 MC78M05CDT, U5 SMF05

Commit message: Version 1.1 Produced
Moved in from archive
Parts:
- removed C4: 560P, Custom Parts:R_0603_sm, symbol C
- removed R6, R7: 4K7, Custom Parts:R_0603_sm, symbol R
- removed U1, U2: MCP2551-I/SN, Power_Integrations:SO-8, symbol MCP2551-I/SN
- added C13, C14: 100N, Custom Parts:R_0603_sm, symbol C
- added CON1: BARREL_JACK, Connect:BARREL_JACK, symbol BARREL_JACK
- added CON2: AVR-JTAG-10, Socket_Strips:Socket_Strip_Straight_2x05, symbol AVR-JTAG-10
- added D1, D4: RED, Custom Parts:Diode_0805_12, symbol LED
- added D2, D5, D6: BLUE, Custom Parts:Diode_0805_12, symbol LED
- added F1, F2: FUSE, Custom Parts:R_1210_SM, symbol FUSE
- added FB1, FB2: 220, Custom Parts:Diode_0805_12_SM, symbol FILTER
- added J1: +5V_SRC, Socket_Strips:Socket_Strip_Straight_1x03, symbol CONN_01X03
- added P1, P2: USB_OTG, Custom Parts:USB_Micro-B-DX4R005JJ2R1800, symbol USB_OTG
- added P3: DIAG Port, Socket_Strips:Socket_Strip_Straight_1x12, symbol CONN_01X12
- added R10, R11, R12, R13, R14, R15, R8: 470, Custom Parts:R_0603_sm, symbol R
- added R9: 4K7, Custom Parts:R_0603_sm, symbol R
- added SW1: SPST, Custom Parts:SW_SPST_FSMSM_SM, symbol SPST
- added U2: FT232RL-SSOP, Housings_SSOP:SSOP-28_5.3x10.2mm_Pitch0.65mm, symbol FT232RL-SSOP
- added U5, U6: MCP25625, Housings_SSOP:SSOP-28_5.3x10.2mm_Pitch0.65mm, symbol MCP25625
- added X1: TXC, Custom Parts:TXC, symbol TXC
- C1, C2: value 560P -> 10N
- C3: value 560P -> 100N
- CON3: renamed from CON?; footprint AVR-AW-6 -> Socket_Strips:Socket_Strip_Straight_2x03
- R1: value 470 -> 22
- R2, R3: value 100 -> 22
- R4, R5: value 100 -> DNS
- U1: renamed from U?; footprint (none) -> Housings_QFP:LQFP-64_10x10mm_Pitch0.5mm
- renumbered C9 to C10, C10 to C11, C11 to C12, C12 to C4, C13 to C5, C5 to C6, C6 to C7, C7 to C8, C8 to C9, D1 to D3, F1 to F3, J1 to J2, J2 to J3, R9 to R6, R8 to R7, U5 to U4
Connections:
- net +12V: now also CON1.1
- net +5V: now also C13.1, C14.1, CON2.4, J1.2 (P2), R10.2, R11.2, R12.2, R13.2, R14.2, R15.2, U2.20 (VCC), U2.4 (VCCIO), U5.1 (VIO), U5.19 (VDD), U5.27 (VDDA), U6.1 (VIO), U6.19 (VDD), U6.27 (VDDA); no longer R1.1
- net CAR_CANH: now also U6.3 (CANL); no longer R5.1
- net CAR_CANL: now also U6.4 (CANH); no longer R4.1
- net GND: now also C13.2, C14.2, CON1.2, CON2.10, CON2.2, D6.1 (K), P1.5 (GND), P1.6 (shield), P2.5 (GND), P2.6 (shield), P3.1 (P1), R9.2, U2.18 (GND), U2.21 (GND), U2.25 (AGND), U2.26 (TEST), U2.7 (GND), U5.10 (GND), U5.26 (VSS), U6.10 (GND), U6.26 (VSS), X1.2 (GND)
- net IVI_CANH: now also U5.3 (CANL); no longer R2.1
- net IVI_CANL: now also U5.4 (CANH); no longer R3.1
- net LOOP_A: now also J3.6 (P6), R7.1, SW1.2; no longer R7.2, U1.47 (PD00)
- net LOOP_B: now also J3.1, R6.1, SW1.1; no longer R6.2, U1.48 (PD01)
- net ~RESET/A_DATA: now also J2.1, CON2.6; no longer J2.6 (P6)
- net at C3.1: now also U2.17 (3V3O); no longer R4.2
- net CLK2_OUT: now reaches R5.2
- net CLK2_OUT: now also U6.22 (CLKOUT)
- net at C2.1: now also F2.2, P2.1 (VCC); no longer R3.2
- net at R2.2: now also R1.2, R3.2, X1.3 (CLK); no longer C1.1
- net +3V3: now reaches C4.1, U1.28 (VDDIN_33)
- net +3V3: now also X1.1 (OE), X1.4 (VDD)
- net TCK: now reaches U1.1 (PA00-TCK)
- net TCK: now also CON2.1
- net TDI: now reaches U1.2 (PA01-TDI)
- net TDI: now also CON2.9
- net VBUS: now reaches U1.23 (VBUS)
- net VBUS: now also FB1.1, J1.3 (P3)
- net USBM: now reaches U1.24 (DM)
- net USBM: now also P1.2 (D-)
- net USBP: now reaches U1.25 (DP)
- net USBP: now also P1.3 (D+)
- net TDO: now reaches U1.3 (PA02-TDO)
- net TDO: now also CON2.3
- net CLK1: now reaches U1.31 (PB30)
- net CLK1: now also R1.1, R4.1
- net IVI_INT: now reaches U1.34 (PC03)
- net IVI_INT: now also U5.13 (~INT)
- net IVI_RESET: now reaches U1.37 (PC04)
- net IVI_RESET: now also U5.18 (~RESET)
- net IVI_STBY: now reaches U1.38 (PC05)
- net IVI_STBY: now also U5.5 (STBY)
- net TMS: now reaches U1.4 (PA03-TMS)
- net TMS: now also CON2.5
- net SCLK: now reaches U1.49 (PD02)
- net SCLK: now also P3.8 (P8), U5.14 (SCK), U6.14 (SCK)
- net CAR_CS: now reaches U1.50 (PD03)
- net CAR_CS: now also P3.6 (P6), U6.17 (~CS)
- net TX_DBG: now reaches U1.53 (PD11)
- net TX_DBG: now also P3.4 (P4), U2.5 (RXD)
- net RX_DBG: now reaches U1.54 (PD12)
- net RX_DBG: now also P3.5 (P5), U2.1 (TXD)
- net CAR_RESET: now reaches U1.55 (PD13)
- net CAR_RESET: now also U6.18 (~RESET)
- net CAR_STBY: now reaches U1.56 (PD14)
- net CAR_STBY: now also U6.5 (STBY)
- net CAR_INT: now reaches U1.57 (PD21)
- net CAR_INT: now also U6.13 (~INT)
- net LED1: now reaches U1.62 (PB00)
- net LED1: now also D4.1 (K)
- net LED2: now reaches U1.63 (PB01)
- net LED2: now also D5.1 (K)
- removed net 5P: J2.1, R1.2, U4.3 (A)
- net RX0: no longer names the net of U1.45 (PC21-CANRX0)
- net RX0: now also R7.2
- net RX1: no longer names the net of U1.39 (PC15-CANRX1)
- net TX0: no longer names the net of U1.46 (PC22-CANTX0)
- net TX0: now also R6.2
- net TX1 renamed IVI_CS
- net IVI_CS: now also P3.7 (P7), U5.17 (~CS)
- new net: J2.6 (P6), R12.1
- new net: D1.1 (K), U2.23 (CBUS0)
- new net: D1.2 (A), R10.1
- new net: D2.1 (K), U2.22 (CBUS1)
- new net: D2.2 (A), R11.1
- new net: F2.1, FB2.2
- new net: R8.1, R9.1, U2.19 (~RESET)
- new net: C1.1, F1.2, P1.1 (VCC)
- new net: F1.1, FB1.2
- new net: D4.2 (A), R13.1
- new net: D5.2 (A), R14.1
- new net: D6.2 (A), R15.1
- new net CAR_Rx0BF: U6.12 (~Rx0BF)
- new net CAR_Rx1BF: U6.11 (~Rx1BF)
- new net CAR_RxCAN: P3.2 (P2), U6.21 (RxCAN), U6.28 (RxD)
- new net CAR_Tx0RTS: U6.23 (~Tx0RTS)
- new net CAR_Tx1RTS: U6.6 (~Tx1RTS)
- new net CAR_Tx2RTS: U6.7 (~Tx2RTS)
- new net CAR_TxCAN: P3.3 (P3), U6.20 (TxCAN), U6.24 (TxD)
- new net CLK2: R2.1, U6.9 (OSC1)
- new net CLK3: R3.1, R5.1, U5.9 (OSC1)
- new net CLK3_OUT: R4.2, U5.22 (CLKOUT)
- new net IVI_Rx0BF: U5.12 (~Rx0BF)
- new net IVI_Rx1BF: U5.11 (~Rx1BF)
- new net IVI_RxCAN: P3.12 (P12), U5.21 (RxCAN), U5.28 (RxD)
- new net IVI_Tx0RTS: U5.23 (~Tx0RTS)
- new net IVI_Tx1RTS: U5.6 (~Tx1RTS)
- new net IVI_Tx2RTS: U5.7 (~Tx2RTS)
- new net IVI_TxCAN: P3.11 (P11), U5.20 (TxCAN), U5.24 (TxD)
- new net MISO: P3.9 (P9), U1.48 (PD01), U5.16 (MISO), U6.16 (MISO)
- new net MOSI: P3.10 (P10), U1.47 (PD00), U5.15 (MOSI), U6.15 (MOSI)
- new net USB+: P2.3 (D+), U2.15 (USBDP)
- new net USB-: P2.2 (D-), U2.16 (USBDM)
- new net USB5: FB2.1, J1.1 (P1), R8.2
Other:
- note added: "RX\n\nTX\n"
- moved on the sheet: C10, C11, C12, C4, C5, C6, C7, C8, C9, CON3, D3, F3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

Commit message: Active project import
moved from archive
Parts:
- added JP1, JP6: Matrix A, Connect:GS3, symbol JUMPER3
- added JP10, JP5: Matrix E, Connect:GS3, symbol JUMPER3
- added JP2, JP7: Matrix B, Connect:GS3, symbol JUMPER3
- added JP3, JP8: Matrix C, Connect:GS3, symbol JUMPER3
- added JP4, JP9: Matrix D, Connect:GS3, symbol JUMPER3
- added R16, R17, R18, R19: 0, Custom Parts:R_0603_sm, symbol R
- added R20, R21: 120, Custom Parts:R_0603_sm, symbol R
- added SW2, SW3: SPST, Custom Parts:SW_SPST_FSMSM_SM, symbol SPST
- C1, C2, C6: Mouser (none) -> 77-VJ0603Y103KXACBC
- C10, C11, C12, C13, C14, C3, C4, C5, C8, C9: Mouser (none) -> 581-06035C104KAT2A
- C7: value 4U7 -> 47U; footprint Capacitors_Tantalum_SMD:TantalC_SizeA_EIA-3216_Reflow -> Capacitors_SMD:c_elec_6.3x5.3; Mouser (none) -> 140-VE470M1ETR0605
- CON1: Mouser (none) -> 502-RAPC722X
- CON2: footprint Socket_Strips:Socket_Strip_Straight_2x05 -> Pin_Headers:Pin_Header_Straight_2x05
- CON3: footprint Socket_Strips:Socket_Strip_Straight_2x03 -> Pin_Headers:Pin_Header_Straight_2x03; Mouser (none) -> 855-M20-9980346
- D1: value RED -> YELLOW; Mouser (none) -> 630-HSMY-C170
- D2: value BLUE -> WHITE; Mouser (none) -> 859-LTW-170ZDC
- D3: footprint Diodes_SMD:Diode-SMB_Standard -> Diodes_SMD:SMB_Handsoldering; Mouser (none) -> 511-SMBJ16A
- D4: Mouser (none) -> 630-HSMH-C170
- D5: value BLUE -> GREEN; Mouser (none) -> 630-HSMG-C170
- D6: Mouser (none) -> 630-HSMR-C170
- F1, F2, F3: Mouser (none) -> 530-0ZCH0050FF2G
- FB1, FB2: Mouser (none) -> 810-MPZ1608S221ATA00
- J1: footprint Socket_Strips:Socket_Strip_Straight_1x03 -> Pin_Headers:Pin_Header_Straight_1x03; Mouser (none) -> 855-M20-9990346
- J2, J3: Mouser (none) -> 523-L77-DE09S
- P1, P2: Mouser (none) -> 656-DX4R005JJ2R1800
- P3: footprint Socket_Strips:Socket_Strip_Straight_1x12 -> Pin_Headers:Pin_Header_Straight_1x12; Mouser (none) -> 855-M20-9991246
- R1, R2, R3: Mouser (none) -> 71-CRCW0603-22.1-E3
- R10, R11, R12, R13, R14, R15, R6, R7, R8: Mouser (none) -> 71-CRCW0603-470-E3
- R4, R5: value DNS -> 470; Mouser (none) -> 71-CRCW0603-470-E3
- R9: Mouser (none) -> 71-CRCW0603-4.7K-E3
- SW1: Mouser (none) -> 653-A6TN-1104
- U1: Mouser (none) -> 556-AT32UC3C2512CA2T
- U2: Mouser (none) -> 895-FT232RL
- U3: Mouser (none) -> 511-L78M05CDT-TR
- U4: Mouser (none) -> 863-SMF05CT2G
- U5, U6: Mouser (none) -> MCP25625-E/SS
- X1: Mouser (none) -> 634-501BAA16M0000CAG
Connections:
- net +5V: no longer C14.1, R10.2, R11.2, U2.20 (VCC), U2.4 (VCCIO)
- net CAR_CANH: now also U6.4 (CANH), R21.2; no longer U6.3 (CANL)
- net CAR_CANL: now also U6.3 (CANL), SW3.2; no longer U6.4 (CANH)
- net CAR_CS: now also P3.4 (P4); no longer P3.6 (P6)
- net CAR_INT: now also U1.60 (PD29); no longer U1.57 (PD21)
- net CAR_RxCAN: now also P3.9 (P9), U1.45 (PC21-CANRX0), R17.1; no longer P3.2 (P2), U6.21 (RxCAN)
- net CAR_TxCAN: now also P3.8 (P8), U1.46 (PC22-CANTX0), R19.1; no longer P3.3 (P3), U6.20 (TxCAN)
- net CLK1: no longer R4.1
- net CLK2_OUT: no longer R5.2
- net CLK3: no longer R5.1
- net CLK3_OUT: no longer R4.2
- net GND: no longer J2.5, J3.5
- net IVI_CANH: now also U5.4 (CANH), R20.2; no longer U5.3 (CANL)
- net IVI_CANL: now also U5.3 (CANL), SW2.2; no longer U5.4 (CANH)
- net IVI_CS: now also P3.10 (P10), U1.41 (PC17); no longer P3.7 (P7), U1.40 (PC16-CANTX1)
- net IVI_RxCAN: now also U1.39 (PC15-CANRX1), R16.1; no longer U5.21 (RxCAN)
- net IVI_TxCAN: now also U1.40 (PC16-CANTX1), R18.1; no longer U5.20 (TxCAN)
- net LED1: now also U1.58 (PD27); no longer U1.62 (PB00)
- net LED2: now also U1.59 (PD28); no longer U1.63 (PB01)
- net LOOP_A: now also JP1.1, JP2.1, JP3.1, JP4.1, JP5.1; no longer J3.6 (P6)
- net LOOP_B: now also JP1.3, JP2.3, JP3.3, JP4.3, JP5.3; no longer J3.1
- net MISO: now also P3.6 (P6); no longer P3.9 (P9)
- net MOSI: now also P3.7 (P7); no longer P3.10 (P10)
- net RX_DBG: now also P3.2 (P2), R4.1; no longer P3.5 (P5), U2.1 (TXD)
- net SCLK: now also P3.5 (P5); no longer P3.8 (P8)
- net TX_DBG: now also P3.3 (P3), R5.1; no longer P3.4 (P4), U2.5 (RXD)
- net USB5: now also C14.1, R10.2, R11.2, U2.20 (VCC), U2.4 (VCCIO)
- net ~RESET/A_DATA: now also JP10.3, JP6.3, JP7.3, JP8.3, JP9.3; no longer J2.1
- net at R7.2: now also U1.43 (PC19); no longer U1.45 (PC21-CANRX0)
- net at J2.6 (P6): no longer R12.1
- net B: now reaches J3.4
- net B: now also JP2.2, JP7.2
- net E: now reaches J3.8 (P8)
- net E: now also JP10.2, JP5.2
- net at R6.2: now also U1.44 (PC20); no longer U1.46 (PC22-CANTX0)
- new net: R19.2, U6.20 (TxCAN)
- new net: R17.2, U6.21 (RxCAN)
- new net: R18.2, U5.20 (TxCAN)
- new net: R16.2, U5.21 (RxCAN)
- new net: JP10.1, JP6.1, JP7.1, JP8.1, JP9.1, R12.1
- new net: R4.2, U2.1 (TXD)
- new net: R5.2, U2.5 (RXD)
- new net: R20.1, SW2.1
- new net: R21.1, SW3.1
- new net A: J3.1, JP1.2, JP6.2
- new net C: J3.5, JP3.2, JP8.2
- new net D: J3.6 (P6), JP4.2, JP9.2
Other:
- moved on the sheet: C1, C10, C11, C12, C13, C14, C2, C3, C6, C7, C8, C9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
